Commit message: ajuste de orientação rplidar

File: description/lidar.xacro (robot description, xacro)
@@ -4,5 +4,5 @@
         <parent link="chassis"/>
         <child link="laser_frame"/>
-        <origin xyz="0.357 0 0.135" rpy="0 0 0"/>
+        <origin xyz="0.357 0 0.135" rpy="0 0 3.14159"/>
     </joint>
     <link name="laser_frame">
@@ -26,5 +26,5 @@
         </collision>
         <xacro:inertial_cylinder mass="0.170" length="0.026" radius="0.035">
-            <origin xyz="0 0 0" rpy="0 0 0"/>
+            <origin xyz="0 0 0" rpy="0 0 3.14159"/>
         </xacro:inertial_cylinder>
     </link>

Commit message: ajustes para geração de modo navegação.

File: description/lidar.xacro (robot description, xacro)
@@ -14,5 +14,5 @@
         </visual>
         <visual>
-            <origin xyz="-0.014 0 -0.019"/>
+            <origin xyz="0.014 0 -0.019"/>
             <geometry>
                 <cylinder radius="0.052" length="0.038"/>
